File: boards/v1.1/PicoFightingBoard.kicad_pcb (KiCad board)
At the start: 2 copper layers, 96.1 x 45.2 mm, 25 parts, among them J5 ST01x05, J6 ST01x05, J7 ST01x05, J8 ST01x05, U1 Pico, U2 SN74LV1T34DBV

Commit message: Commit latest rev
Parts:
- removed  : , FeralAI:GS_Ground_back
- removed  : , FeralAI:GS_Ground (x5)
- removed PLEDS: Conn_01x05_Male, Connector_JST:JST_PH_S5B-PH-K_1x05_P2.00mm_Horizontal
- removed the RGB LEDS at (108.1, 93.5)
- added G***: LOGO, FeralAI:PFB_Logo, F.Cu at (130.7, 99.4)
- added J12: Conn_01x04_Male, Connector_JST:JST_PH_S4B-PH-K_1x04_P2.00mm_Horizontal, F.Cu at (108.6, 107.5)
- added PGM BUTTONS: Conn_01x04_Male, Connector_JST:JST_PH_S4B-PH-K_1x04_P2.00mm_Horizontal, F.Cu at (170.2, 120.1)
- added PLAYER LEDS: Conn_01x05_Male, Connector_JST:JST_PH_S5B-PH-K_1x05_P2.00mm_Horizontal, F.Cu at (146.3, 120.1)
- added R5: 330, Resistor_SMD:R_0805_2012Metric, F.Cu at (113.3, 90.3)
- added RESET BUTTON: Conn_01x02_Male, Connector_PinHeader_2.54mm:PinHeader_1x02_P2.54mm_Vertical, F.Cu at (184.3, 120.1)
- added RGB LEDS: Conn_01x04_Male, Connector_JST:JST_PH_S4B-PH-K_1x04_P2.00mm_Horizontal, F.Cu at (108.6, 93.0)
- J5, J6, J7, J8: footprint TerminalBlock_Phoenix:TerminalBlock_Phoenix_PT-1,5-5-3.5-H_1x05_P3.50mm_Horizontal -> FeralAI:TerminalBlock_Phoenix_PT-1,5-5-3.5-H_1x05_P3.50mm_Horizontal
- J9: renamed from STEMMA QT
- moved J5 14.0 mm to (129.5, 82.5), turned to 180 degrees
- moved J6 14.0 mm to (147.3, 82.5), turned to 180 degrees
- moved J7 14.0 mm to (165.1, 82.5), turned to 180 degrees
- moved J8 14.0 mm to (182.9, 82.5), turned to 180 degrees
- moved R1 9.41 mm to (139.1, 114.9)
- moved R2 9.41 mm to (141.1, 114.9)
- moved R3 9.41 mm to (143.1, 114.9)
- moved R4 9.41 mm to (145.2, 114.9)
- moved J9 7.64 mm to (116.3, 110.5)
- moved U2 6.62 mm to (117.9, 91.4)
Connections:
- J5 pad 1: /GND -> /1K
- J5 pad 2: /4K -> /2K
- J5 pad 4: /2K -> /4K
- J5 pad 5: /1K -> /GND
- J6 pad 1: /GND -> /1P
- J6 pad 2: /4P -> /2P
- J6 pad 4: /2P -> /4P
- J6 pad 5: /1P -> /GND
- J7 pad 1: /START -> /GND
- J7 pad 2: /SELECT -> /GND
- J7 pad 4: /GND -> /SELECT
- J7 pad 5: /GND -> /START
- J8 pad 1: /RIGHT -> /5V
- J8 pad 2: /LEFT -> /DOWN
- J8 pad 4: /DOWN -> /LEFT
- J8 pad 5: /5V -> /RIGHT
- J9 pad 1: /GND -> /SCL
- J9 pad 2: /3V3 -> /SDA
- J9 pad 3: /SDA -> /3V3
- J9 pad 4: /SCL -> /GND
- U1 pad 13: Net-(U1-Pad13) -> /GND
- U1 pad 18: Net-(U1-Pad18) -> /GND
- U1 pad 21: /SDA -> /PLED1
- U1 pad 22: /SCL -> /PLED2
- U1 pad 23: Net-(U1-Pad23) -> /GND
- U1 pad 24: /PLED1 -> /PLED3
- U1 pad 25: /PLED2 -> /PLED4
- U1 pad 26: /PLED3 -> /TP
- U1 pad 27: /PLED4 -> /LSB
- U1 pad 28: Net-(U1-Pad28) -> /GND
- U1 pad 29: /TP -> /RSB
- U1 pad 31: /LSB -> /SDA
- U1 pad 32: /RSB -> /SCL
- U1 pad 33: Net-(U1-Pad33) -> /GND
- U1 pad 34: Net-(U1-Pad34) -> /SETTINGS
- U1 pad 8: Net-(U1-Pad8) -> /GND
- U2 pad 4: /RGB_5V_DATA -> /RGB_DATA_5V
Routing:
- net /SCL: track 43.3 -> 113.0 mm
- net /SDA: track 40.9 -> 105.0 mm
- net /1P: track 81.6 -> 116.7 mm
- net Net-(J2-Pad9): track 35.1 -> 0.02 mm
- net /RUN: track 0.00 -> 26.8 mm
- net /3V3: track 87.9 -> 106.3 mm
- net /SETTINGS: track 0.00 -> 12.7 mm
- net Net-(J3-Pad5): track 2.42 -> 11.4 mm
- net /PLED3: track 12.1 -> 21.0 mm
- net Net-(J3-Pad4): track 2.41 -> 11.2 mm
- net Net-(J3-Pad3): track 2.39 -> 11.1 mm
- net Net-(J3-Pad2): track 2.40 -> 11.1 mm
- net /RGB_DATA_5V: track 0.00 -> 7.89 mm
- net /PLED4: track 12.6 -> 20.0 mm
- net /LSB: track 17.6 -> 10.7 mm
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- added copper zone on B.Cu, net (none)
- added copper zone on F.Cu, net (none)
Other:
- board text added: "3V"
- board text added: "DOWN"
- board text added: "EXP. PORTS"
- board text added: "FN1"
- board text added: "FN2"
- board text added: "FN3"
- board text added: "GND"
- board text added: "HOME"
- board text added: "LEFT"
- board text added: "LS"
- board text added: "PFB-20211204"
- board text added: "RESET BUTTON DOUBLE PRESS QUICKLY FOR FLASH MODE"
- board text added: "RIGHT"
- board text added: "RS"
- board text added: "RUN"
- board text added: "RX"
- board text added: "SELECT"
- board text added: "START"
- board text added: "TP"
- board text added: "TX"
- board text added: "UP"
- board text added: "v1.1"
- board text removed: "A2"
- board text removed: "HOM"
- board text removed: "L3"
- board text removed: "Pico Fighting Board"
- board text removed: "R3"
- board text removed: "SEL"
- board text removed: "STA"
- board text removed: "VCC"
- board text removed: "v1.1 20211203"
- board text removed: "▲"
- board text removed: "▶"
- board text removed: "▶▶▶"
- board text removed: "▼"
- board text removed: "◀"

Commit message: Almost there
Parts:
- added DEBUG: Conn_01x04_Male, Connector_JST:JST_SH_BM04B-SRSS-TB_1x04-1MP_P1.00mm_Vertical, F.Cu at (142.6, 101.6)
- added G***: LOGO, FeralAI:DesignedBy, F.Cu at (127.6, 110.4)
- added G***: LOGO, FeralAI:FeralAI, F.Cu at (127.9, 112.7)
- J10: renamed from RESET BUTTON
- moved G*** 2.54 mm to (128.2, 100.1)
- renumbered J12 to JST-PH, U1 to PICO, J9 to QWIIC
Connections:
- PICO pad 11: /1P -> /2P
- PICO pad 41: Net-(U1-Pad41) -> /SWCLK
- PICO pad 42: Net-(U1-Pad42) -> /GND
- PICO pad 43: Net-(U1-Pad43) -> /SWDIO
- PLAYER LEDS pad 2: Net-(J3-Pad2) -> /PLED1
- PLAYER LEDS pad 3: Net-(J3-Pad3) -> /PLED2
- PLAYER LEDS pad 4: Net-(J3-Pad4) -> /PLED3
- PLAYER LEDS pad 5: Net-(J3-Pad5) -> /PLED4
- R1 pad 2: Net-(J3-Pad2) -> /PLED1
- R2 pad 2: Net-(J3-Pad3) -> /PLED2
- R3 pad 2: Net-(J3-Pad4) -> /PLED3
- R4 pad 2: Net-(J3-Pad5) -> /PLED4
Routing:
- net /3V3: track 106.3 -> 158.6 mm
- net /2P: track 44.0 -> 79.1 mm
- net /1P: track 116.7 -> 81.6 mm
- net Net-(J3-Pad5): track 11.4 -> 0.00 mm
- net /PLED4: track 20.0 -> 31.4 mm
- net Net-(J3-Pad4): track 11.2 -> 0.00 mm
- net /PLED3: track 21.0 -> 32.2 mm
- net Net-(J3-Pad3): track 11.1 -> 0.00 mm
- net /PLED2: track 17.8 -> 28.9 mm
- net Net-(J3-Pad2): track 11.1 -> 0.00 mm
- net /PLED1: track 12.5 -> 23.6 mm
- net /SWCLK: track 0.00 -> 10.6 mm
- net /GND: track 20.2 -> 25.8 mm
- net /SWDIO: track 0.00 -> 5.37 mm
Other:
- board text added: "EXPANSION 3.3V ONLY"
- board text added: "v1.1-20211204"
- board text removed: "EXP. PORTS"
- board text removed: "PFB-20211204"
- board text removed: "v1.1"

Commit message: Latest v1.1 rev
Parts:
- added C1: 0.1uF, Capacitor_SMD:C_0805_2012Metric, F.Cu at (115.5, 93.0)
- added R6: 4.7k, Resistor_SMD:R_0805_2012Metric, F.Cu at (112.2, 114.8)
- added R7: 4.7k, Resistor_SMD:R_0805_2012Metric, F.Cu at (115.6, 114.8)
- moved QWIIC 2.49 mm to (116.3, 108.0)
- moved JST-PH 2.47 mm to (108.6, 105.0)
- moved R5 2.35 mm to (115.5, 91.0)
- moved RGB LEDS 1.98 mm to (108.6, 91.0)
- moved U2 1.73 mm to (119.2, 90.3)
- renumbered DEBUG to J13, PICO to U1
Routing:
- net /3V3: track 158.6 -> 188.1 mm, vias 0 -> 1
- net /SCL: track 113.0 -> 95.1 mm
- net /SDA: track 105.0 -> 89.7 mm
- net /GND: track 25.8 -> 33.3 mm
- net /UP: track 91.4 -> 96.3 mm
- net /3K: track 78.8 -> 82.9 mm
- net /DOWN: track 87.5 -> 90.2 mm
- net /3P: track 82.3 -> 85.0 mm
- net /LEFT: track 100.1 -> 102.7 mm
- net /1K: track 79.9 -> 82.5 mm
- net /1P: track 81.6 -> 84.2 mm
- net /4P: track 76.9 -> 79.4 mm
- net /RIGHT: track 85.6 -> 88.1 mm
- net /START: track 79.9 -> 82.4 mm
- net /SELECT: track 83.0 -> 85.5 mm
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- removed copper zone on B.Cu, net (none)
- removed copper zone on F.Cu, net (none)
Other:
- board text added: "EXPANSION (3.3V)"
- board text removed: "EXPANSION 3.3V ONLY"
