File: boards/v1.1/PicoFightingBoard.kicad_pcb (KiCad board)
At the start: 2 copper layers, 96.1 x 45.2 mm, 26 parts, among them J1 Conn_01x04_Male, J10 Conn_01x02_Male, J11 Conn_01x04_Male, J12 Conn_01x04_Male, J13 Conn_01x04_Male, J2 Conn_02x10_Odd_Even, J3 Conn_01x05_Male, J4 Conn_01x04_Male, J5 ST01x05, J6 ST01x05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

Commit message: Update v1.1
Parts:
- removed the G*** at (127.9, 111.2)
- added H1: MountingHole, MountingHole:MountingHole_2.7mm_M2.5, F.Cu at (107.0, 82.8)
- added H2: MountingHole, MountingHole:MountingHole_2.7mm_M2.5, F.Cu at (196.0, 82.9)
- added H3: MountingHole, MountingHole:MountingHole_2.7mm_M2.5, F.Cu at (107.1, 121.0)
- added H4: MountingHole, MountingHole:MountingHole_2.7mm_M2.5, F.Cu at (196.0, 120.8)
- J13, J9: footprint Connector_JST:JST_SH_BM04B-SRSS-TB_1x04-1MP_P1.00mm_Vertical -> FeralAI:BOOM_SH_C145961_1x04_P1.00mm_Vertical
- moved G*** 2.53 mm to (129.6, 111.7)
- moved G*** 0.96 mm to (128.9, 99.9)
- moved R6 0.33 mm to (112.5, 114.8)
Connections:
- J1 pad 1: /RGB_DATA_5V -> Net-(J1-Pad1)
- J3 pad 2: /PLED1 -> Net-(J3-Pad2)
- J3 pad 3: /PLED2 -> Net-(J3-Pad3)
- J3 pad 4: /PLED3 -> Net-(J3-Pad4)
- J3 pad 5: /PLED4 -> Net-(J3-Pad5)
- R1 pad 2: /PLED1 -> Net-(J3-Pad2)
- R2 pad 2: /PLED2 -> Net-(J3-Pad3)
- R3 pad 2: /PLED3 -> Net-(J3-Pad4)
- R4 pad 2: /PLED4 -> Net-(J3-Pad5)
- R5 pad 2: /RGB_DATA_5V -> Net-(J1-Pad1)
Routing:
- net Net-(J3-Pad5): track 0.00 -> 11.4 mm
- net /PLED4: track 31.4 -> 20.0 mm
- net /PLED3: track 32.5 -> 21.3 mm
- net Net-(J3-Pad4): track 0.00 -> 11.2 mm
- net /PLED2: track 26.7 -> 15.5 mm
- net Net-(J3-Pad3): track 0.00 -> 11.1 mm
- net /PLED1: track 25.2 -> 14.0 mm
- net Net-(J3-Pad2): track 0.00 -> 11.1 mm
- net Net-(J1-Pad1): track 0.00 -> 6.04 mm
- net /RGB_DATA_5V: track 8.44 -> 2.39 mm
- net /SCL: track 95.1 -> 99.2 mm
- net /3V3: track 188.1 -> 191.9 mm, vias 1 -> 2
- net /SDA: track 89.7 -> 93.4 mm
- net /SWDIO: track 5.37 -> 8.08 mm
- net /SWCLK: track 10.6 -> 12.8 mm
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Other:
- board text added: "DESIGNED BY"
- board text added: "I2C EXPANSION"
- board text added: "OPT BUTTONS"
- board text added: "SCL"
- board text added: "SDA"
- board text removed: "EXPANSION (3.3V)"
- board text removed: "JST-PH"
- board text removed: "PGM BUTTONS"
- board text removed: "RX"
- board text removed: "TX"
