File: boards/v1.1/PicoFightingBoard.sch (KiCad schematic (older format))
At the start: 15 parts, among them J1 Conn_01x03_Male, J2 Conn_02x10_Odd_Even, J3 Conn_01x05_Male, J4 Conn_01x04_Male, J5 ST01x05, J6 ST01x05, J7 ST01x05, J8 ST01x05, J9 Conn_01x04_Male, U1 Pico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

Commit message: Commit latest rev
Parts:
- removed J1: Conn_01x03_Male, Connector_PinHeader_2.54mm:PinHeader_1x03_P2.54mm_Vertical, symbol Connector:Conn_01x03_Male
- added J1, J11, J12: Conn_01x04_Male, Connector_JST:JST_PH_S4B-PH-K_1x04_P2.00mm_Horizontal, symbol Connector:Conn_01x04_Male
- added J10: Conn_01x02_Male, Connector_PinHeader_2.54mm:PinHeader_1x02_P2.54mm_Vertical, symbol Connector:Conn_01x02_Male
- added R5: 330, Resistor_SMD:R_0805_2012Metric, symbol Device:R
- J5, J6, J7, J8: footprint TerminalBlock_Phoenix:TerminalBlock_Phoenix_PT-1,5-5-3.5-H_1x05_P3.50mm_Horizontal -> TerminalBlock_MetzConnect:TerminalBlock_MetzConnect_Type059_RT06305HBWC_1x05_P3.50mm_Horizontal
Connections:
- net labels added: RGB_DATA_5V, SETTINGS
- net labels removed: RGB_5V_DATA
- wire segments 93 -> 113
Other:
- moved on the sheet: J2, J3, J4, J5, J6, J7, J8, J9, R1, R2, R3, R4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

Commit message: Almost there
Parts:
- added J13: Conn_01x04_Male, Connector_JST:JST_SH_BM04B-SRSS-TB_1x04-1MP_P1.00mm_Vertical, symbol Connector:Conn_01x04_Male
Connections:
- net labels added: SWCLK, SWDIO
- wire segments 113 -> 120
Other:
- moved on the sheet: R1, R2, R3, R4
Changed lines of the file:
@@
 L Device:R R1
 U 1 1 614D343B
-P 5500 6450
-F 0 "R1" H 5570 6496 50  0000 L CNN
-F 1 "330" H 5570 6405 50  0000 L CNN
-F 2 "Resistor_SMD:R_0805_2012Metric" V 5430 6450 50  0001 C CNN
-F 3 "~" H 5500 6450 50  0001 C CNN
-	1    5500 6450
+P 5800 6450
+F 0 "R1" H 5870 6496 50  0000 L CNN
+F 1 "330" H 5870 6405 50  0000 L CNN
+F 2 "Resistor_SMD:R_0805_2012Metric" V 5730 6450 50  0001 C CNN
+F 3 "~" H 5800 6450 50  0001 C CNN
+	1    5800 6450
 	0    1    1    0
 $EndComp
@@
 L Device:R R2
 U 1 1 614D5962
-P 5500 6550
-F 0 "R2" H 5570 6596 50  0000 L CNN
-F 1 "330" H 5570 6505 50  0000 L CNN
-F 2 "Resistor_SMD:R_0805_2012Metric" V 5430 6550 50  0001 C CNN
-F 3 "~" H 5500 6550 50  0001 C CNN
-	1    5500 6550
+P 5800 6550
+F 0 "R2" H 5870 6596 50  0000 L CNN
+F 1 "330" H 5870 6505 50  0000 L CNN
+F 2 "Resistor_SMD:R_0805_2012Metric" V 5730 6550 50  0001 C CNN
+F 3 "~" H 5800 6550 50  0001 C CNN
+	1    5800 6550
 	0    1    1    0
 $EndComp
-Wire Wire Line
-	5300 6450 5350 6450
-Wire Wire Line
-	5300 6550 5350 6550
-Wire Wire Line
-	5300 6650 5350 6650
-Wire Wire Line
-	5300 6750 5350 6750
 $Comp
 L Connector:Screw_Terminal_01x05 J5
@@
 1P
 Text Label 4775 2575 0    50   ~ 0
-1P
+2P
 Text Label 4775 2675 0    50   ~ 0
 3P
@@
 3V3
 Wire Wire Line
-	5975 6450 5650 6450
-Wire Wire Line
-	5975 6550 5650 6550
-Wire Wire Line
-	5975 6650 5650 6650
-Wire Wire Line
-	5975 6750 5650 6750
-Text Label 5675 6450 0    50   ~ 0
+	6275 6450 5950 6450
+Wire Wire Line
+	6275 6550 5950 6550
+Wire Wire Line
+	6275 6650 5950 6650
+Wire Wire Line
+	6275 6750 5950 6750
+Text Label 5975 6450 0    50   ~ 0
 PLED1
-Text Label 5675 6550 0    50   ~ 0
+Text Label 5975 6550 0    50   ~ 0
 PLED2
-Text Label 5675 6650 0    50   ~ 0
+Text Label 5975 6650 0    50   ~ 0
 PLED3
-Text Label 5675 6750 0    50   ~ 0
+Text Label 5975 6750 0    50   ~ 0
 PLED4
 Wire Wire Line
@@
 L Device:R R3
 U 1 1 614D616C
-P 5500 6650
-F 0 "R3" H 5570 6696 50  0000 L CNN
-F 1 "330" H 5570 6605 50  0000 L CNN
-F 2 "Resistor_SMD:R_0805_2012Metric" V 5430 6650 50  0001 C CNN
-F 3 "~" H 5500 6650 50  0001 C CNN
-	1    5500 6650
+P 5800 6650
+F 0 "R3" H 5870 6696 50  0000 L CNN
+F 1 "330" H 5870 6605 50  0000 L CNN
+F 2 "Resistor_SMD:R_0805_2012Metric" V 5730 6650 50  0001 C CNN
+F 3 "~" H 5800 6650 50  0001 C CNN
+	1    5800 6650
 	0    1    1    0
 $EndComp
@@
 L Device:R R4
 U 1 1 614D640B
-P 5500 6750
-F 0 "R4" H 5570 6796 50  0000 L CNN
-F 1 "330" H 5570 6705 50  0000 L CNN
-F 2 "Resistor_SMD:R_0805_2012Metric" V 5430 6750 50  0001 C CNN
-F 3 "~" H 5500 6750 50  0001 C CNN
-	1    5500 6750
+P 5800 6750
+F 0 "R4" H 5870 6796 50  0000 L CNN
+F 1 "330" H 5870 6705 50  0000 L CNN
+F 2 "Resistor_SMD:R_0805_2012Metric" V 5730 6750 50  0001 C CNN
+F 3 "~" H 5800 6750 50  0001 C CNN
+	1    5800 6750
 	0    1    1    0
 $EndComp
@@
 Text Label 7950 5175 0    50   ~ 0
 GND
+Wire Wire Line
+	5300 6450 5650 6450
+Wire Wire Line
+	5300 6550 5650 6550
+Wire Wire Line
+	5300 6650 5650 6650
+Wire Wire Line
+	5300 6750 5650 6750
+Text Label 5350 6450 0    50   ~ 0
+PLED1
+Text Label 5350 6550 0    50   ~ 0
+PLED2
+Text Label 5350 6650 0    50   ~ 0
+PLED3
+Text Label 5350 6750 0    50   ~ 0
+PLED4
+$Comp
+L Connector:Conn_01x04_Male J13
+U 1 1 61AFA94A
+P 3500 4250
+F 0 "J13" H 3775 4650 50  0000 C CNN
+F 1 "Conn_01x04_Male" H 3750 4550 50  0000 C CNN
+F 2 "Connector_JST:JST_SH_BM04B-SRSS-TB_1x04-1MP_P1.00mm_Vertical" H 3500 4250 50  0001 C CNN
+F 3 "~" H 3500 4250 50  0001 C CNN
+	1    3500 4250
+	1    0    0    -1
+$EndComp
+Wire Wire Line
+	5625 3675 5625 3950
+Wire Wire Line
+	5725 3675 5725 3950
+Wire Wire Line
+	5825 3675 5825 3950
+Text Label 5625 3950 1    50   ~ 0
+SWCLK
+Text Label 5725 3950 1    50   ~ 0
+GND
+Text Label 5825 3950 1    50   ~ 0
+SWDIO
+Wire Wire Line
+	4075 4150 3700 4150
+Wire Wire Line
+	4075 4250 3700 4250
+Wire Wire Line
+	4075 4350 3700 4350
+Wire Wire Line
+	3700 4450 4075 4450
+Text Label 3750 4250 0    50   ~ 0
+SWCLK
+Text Label 3750 4150 0    50   ~ 0
+SWDIO
+Text Label 3750 4350 0    50   ~ 0
+3V3
+Text Label 3750 4450 0    50   ~ 0
+GND
 $EndSCHEMATC

Commit message: Latest v1.1 rev
Parts:
- added C1: 0.1uF, Capacitor_SMD:C_0805_2012Metric, symbol Device:C
- added R6, R7: 4.7k, Resistor_SMD:R_0805_2012Metric, symbol Device:R
Connections:
- wire segments 120 -> 126
Changed lines of the file:
@@
 	6725 1775 6425 1775
-Wire Wire Line
-	6725 1975 6425 1975
 Wire Wire Line
 	6725 2675 6425 2675
@@
 Text Label 3750 4450 0    50   ~ 0
 GND
+$Comp
+L Device:C C1
+U 1 1 61AD43CD
+P 10400 5175
+F 0 "C1" H 10515 5221 50  0000 L CNN
+F 1 "0.1uF" H 10515 5130 50  0000 L CNN
+F 2 "Capacitor_SMD:C_0805_2012Metric" H 10438 5025 50  0001 C CNN
+F 3 "~" H 10400 5175 50  0001 C CNN
+	1    10400 5175
+	1    0    0    -1
+$EndComp
+Wire Wire Line
+	9550 5475 10400 5475
+Wire Wire Line
+	10400 5475 10400 5325
+Connection ~ 9550 5475
+Wire Wire Line
+	9550 4775 10400 4775
+Wire Wire Line
+	10400 4775 10400 5025
+$Comp
+L Device:R R7
+U 1 1 61AE3E8D
+P 6875 2475
+F 0 "R7" V 6875 2775 50  0000 L CNN
+F 1 "4.7k" V 6875 2925 50  0000 L CNN
+F 2 "Resistor_SMD:R_0805_2012Metric" V 6805 2475 50  0001 C CNN
+F 3 "~" H 6875 2475 50  0001 C CNN
+	1    6875 2475
+	0    1    1    0
+$EndComp
+$Comp
+L Device:R R6
+U 1 1 61AE5D26
+P 6875 2375
+F 0 "R6" V 6875 2675 50  0000 L CNN
+F 1 "4.7k" V 6875 2825 50  0000 L CNN
+F 2 "Resistor_SMD:R_0805_2012Metric" V 6805 2375 50  0001 C CNN
+F 3 "~" H 6875 2375 50  0001 C CNN
+	1    6875 2375
+	0    1    1    0
+$EndComp
+Wire Wire Line
+	7025 1975 7025 2375
+Wire Wire Line
+	6425 1975 7025 1975
+Wire Wire Line
+	7025 2375 7025 2475
+Connection ~ 7025 2375
 $EndSCHEMATC
