File: boards/v1.1a/PicoFightingBoard.kicad_pcb (KiCad board)
At the start: 2 copper layers, 96.1 x 45.2 mm, 29 parts, among them J1 Conn_01x04_Male, J10 Conn_01x02_Male, J11 Conn_01x04_Male, J12 Conn_01x04_Male, J13 Conn_01x04_Male, J2 Conn_02x10_Odd_Even, J3 Conn_01x05_Male, J4 Conn_01x04_Male, J5 ST01x05, J6 ST01x05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

Commit message: Update to KiCad 6.0.0 for v1.1a board
Other:
- net class Default removed

Commit message: v1.1a final?!?
Parts:
- moved R6 10.1 mm to (121.5, 110.2), turned to 180 degrees
- moved R7 8.99 mm to (121.5, 108.0), turned to 180 degrees
- moved G*** 2.02 mm to (131.5, 111.4)
- moved G*** 0.71 mm to (129.2, 98.9)
- moved U2 0.52 mm to (119.7, 90.3)
- moved H3 0.20 mm to (107.4, 120.7)
- moved H2 0.20 mm to (195.7, 83.2)
- moved H4 0.20 mm to (195.7, 120.5)
- moved H1 0.14 mm to (107.3, 83.1)
Connections:
- U1 pad 35: Net-(U1-Pad35) -> unconnected-(U1-Pad35)
- U1 pad 37: Net-(U1-Pad37) -> unconnected-(U1-Pad37)
- U1 pad 39: Net-(U1-Pad39) -> unconnected-(U1-Pad39)
- U2 pad 1: Net-(U2-Pad1) -> unconnected-(U2-Pad1)
Routing:
- net /3V3: track 191.9 -> 144.4 mm, vias 2 -> 1
- net /SCL: track 99.2 -> 83.7 mm
- net /SDA: track 93.4 -> 83.2 mm
- net /UP: track 96.3 -> 92.4 mm
- net /LEFT: track 102.7 -> 99.5 mm
- net /PLED2: track 15.5 -> 13.0 mm
- net /3P: track 85.0 -> 83.0 mm
- net /1K: track 82.5 -> 80.6 mm
- net /DOWN: track 90.2 -> 88.3 mm
- net /2K: track 85.9 -> 84.0 mm
- net /4P: track 79.4 -> 77.5 mm
- net /1P: track 84.2 -> 82.3 mm
- net /3K: track 82.9 -> 81.1 mm
- net /2P: track 81.5 -> 79.8 mm
- net /START: track 82.4 -> 80.6 mm
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Other:
- board text added: "v1.1a-20220102"
- board text removed: "v1.1a-20211231"
