File: boards/v1.1a/PicoFightingBoard.kicad_sch (KiCad schematic)
At the start: 28 parts, among them J1 Conn_01x04_Male, J10 Conn_01x02_Male, J11 Conn_01x04_Male, J12 Conn_01x04_Male, J13 Conn_01x04_Male, J14 Screw_Terminal_01x04, J2 Conn_02x10_Odd_Even, J3 Conn_01x05_Male, J4 Conn_01x04_Male, J5 Screw_Terminal_01x04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

Commit message: v1.1a final?!?
Parts:
- removed J14, J5, J6, J7, J8: Screw_Terminal_01x04, FeralAI:CONN-TH_DB125-3.5-4P-GN, symbol Connector:Screw_Terminal_01x04
- added J5, J6, J7, J8: ST01x05, TerminalBlock_MetzConnect:TerminalBlock_MetzConnect_Type059_RT06305HBWC_1x05_P3.50mm_Horizontal, symbol Connector:Screw_Terminal_01x05
Connections:
- net 1K: now also J5.1 (Pin_1)
- net 1P: now also J6.1 (Pin_1)
- net 2K: now also J5.2 (Pin_2)
- net 2P: now also J6.2 (Pin_2)
- net 3K: now also J5.3 (Pin_3)
- net 3P: now also J6.3 (Pin_3)
- net 4K: now also J5.4 (Pin_4)
- net 4P: now also J6.4 (Pin_4)
- net 5V: now also J8.1 (Pin_1)
- net DOWN: now also J8.2 (Pin_2)
- net GND: now also J5.5 (Pin_5), J6.5 (Pin_5), J7.1 (Pin_1), J7.2 (Pin_2)
- net HOME: now also J7.3 (Pin_3)
- net LEFT: now also J8.4 (Pin_4)
- net RIGHT: now also J8.5 (Pin_5)
- net SELECT: now also J7.4 (Pin_4)
- net START: now also J7.5 (Pin_5)
- net UP: now also J8.3 (Pin_3)
